File: KiCAD/Capacitor Board/Capacitor Board.kicad_pcb (KiCad board)
At the start: 6 copper layers, 69.7 x 89.6 mm, 9 parts

Commit message: cap board done?
Parts:
- moved C1 0.10 mm to (70.0, 58.8)
- moved C2 0.10 mm to (82.0, 58.8)
- moved C3 0.10 mm to (94.0, 58.8)
- moved C4 0.10 mm to (106.0, 58.8)
Changed lines of the file:
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@@
 	(footprint "Inverter Power Components:CAP_B58035U-FA10_TDK"
 		(layer "F.Cu")
-		(at 82 58.9)
+		(at 82 58.8)
 		(tags "B58035U5106M001 ")
 		(property "Reference" "C2"
@@
 			(polygon
 				(pts
-					(xy 79.5489 43.4568) (xy 84.4511 43.4568) (xy 84.4511 74.3432) (xy 79.5489 74.3432)
+					(xy 79.5489 43.3568) (xy 84.4511 43.3568) (xy 84.4511 74.2432) (xy 79.5489 74.2432)
 				)
 			)
@@
 	(footprint "Inverter Power Components:CAP_B58035U-FA10_TDK"
 		(layer "F.Cu")
-		(at 70 58.9 180)
+		(at 70 58.8 180)
 		(tags "B58035U5106M001 ")
 		(property "Reference" "C1"
@@
 			(polygon
 				(pts
-					(xy 72.4511 74.3432) (xy 67.5489 74.3432) (xy 67.5489 43.4568) (xy 72.4511 43.4568)
+					(xy 72.4511 74.2432) (xy 67.5489 74.2432) (xy 67.5489 43.3568) (xy 72.4511 43.3568)
 				)
 			)
@@
 	(footprint "Inverter Power Components:CAP_B58035U-FA10_TDK"
 		(layer "F.Cu")
-		(at 94 58.9 180)
+		(at 94 58.8 180)
 		(tags "B58035U5106M001 ")
 		(property "Reference" "C3"
@@
 			(polygon
 				(pts
-					(xy 96.4511 74.3432) (xy 91.5489 74.3432) (xy 91.5489 43.4568) (xy 96.4511 43.4568)
+					(xy 96.4511 74.2432) (xy 91.5489 74.2432) (xy 91.5489 43.3568) (xy 96.4511 43.3568)
 				)
 			)
@@
 	(footprint "Inverter Power Components:CAP_B58035U-FA10_TDK"
 		(layer "F.Cu")
-		(at 106 58.9)
+		(at 106 58.8)
 		(tags "B58035U5106M001 ")
 		(property "Reference" "C4"
@@
 			(polygon
 				(pts
-					(xy 103.5489 43.4568) (xy 108.4511 43.4568) (xy 108.4511 74.3432) (xy 103.5489 74.3432)
+					(xy 103.5489 43.3568) (xy 108.4511 43.3568) (xy 108.4511 74.2432) (xy 103.5489 74.2432)
 				)
 			)
@@
 	)
 	(gr_rect
-		(start 64.5958 35.8)
-		(end 67.5 74.4)
+		(start 64.5958 35.7)
+		(end 67.5 74.3)
 		(stroke
 			(width 0.2)
@@
 	)
 	(gr_rect
-		(start 108.5 35.8)
-		(end 111.4042 74.4)
+		(start 108.5 35.7)
+		(end 111.4042 74.3)
 		(stroke
 			(width 0.2)
@@
 		(layer "F.Cu")
 		(net 1)
+	)
+	(gr_poly
+		(pts
+			(xy 72.4958 93.775) (xy 77.7479 99.8375) (xy 82.2521 92.1625) (xy 77 86.1)
+		)
+		(stroke
+			(width 0.2)
+			(type solid)
+		)
+		(fill yes)
+		(layer "F.Cu")
+		(net 2)
+	)
+	(gr_rect
+		(start 72.4958 93.775)
+		(end 79.5 128.9)
+		(stroke
+			(width 0.2)
+			(type solid)
+		)
+		(fill yes)
+		(layer "F.Cu")
+		(net 2)
 	)
 	(gr_rect
@@
 	)
 	(gr_rect
-		(start 72.4 77)
+		(start 75 77)
 		(end 103.6 95.2)
 		(stroke
@@
 	)
 	(gr_rect
-		(start 96.5 56.6)
+		(start 55.1 87)
+		(end 67.1 92.4)
+		(stroke
+			(width 0)
+			(type solid)
+		)
+		(fill yes)
+		(layer "F.Cu")
+		(net 4)
+	)
+	(gr_rect
+		(start 96.5 43.3)
 		(end 103.5042 128.9)
 		(stroke
@@
 	)
 	(gr_rect
-		(start 64.5 35.7)
-		(end 111.5 40.7)
+		(start 54.8 43.3)
+		(end 61.8 128.9)
+		(stroke
+			(width 0.2)
+			(type solid)
+		)
+		(fill yes)
+		(layer "F.Cu")
+		(net 4)
+	)
+	(gr_rect
+		(start 64.5 35.6)
+		(end 111.5 40.6)
 		(stroke
 			(width 0)
@@
 	)
 	(gr_rect
-		(start 72.5 56.6)
-		(end 79.5042 128.9)
+		(start 72.5 43.3)
+		(end 79.5042 82.55)
 		(stroke
 			(width 0.2)
@@
 	)
 	(gr_rect
-		(start 84.4979 35.8)
-		(end 91.5021 74.3)
+		(start 84.4979 35.7)
+		(end 91.5021 74.2)
 		(stroke
 			(width 0.2)
@@
 	)
 	(gr_rect
+		(start 62.2 40.9)
+		(end 64.2 76.7)
+		(stroke
+			(width 0)
+			(type solid)
+		)
+		(fill yes)
+		(layer "F.SilkS")
+	)
+	(gr_rect
 		(start 64.5 95.5)
 		(end 111.5 97.5)
@@
 	)
 	(gr_rect
-		(start 64.5 41)
-		(end 111.5 43)
+		(start 62.2 95.5)
+		(end 64.2 131.3)
+		(stroke
+			(width 0)
+			(type solid)
+		)
+		(fill yes)
+		(layer "F.SilkS")
+	)
+	(gr_rect
+		(start 64.5 40.9)
+		(end 111.5 42.9)
 		(stroke
 			(width 0)
@@
 		(layer "Dwgs.User")
 		(pts
-			(xy 112 31.4) (xy 112.5 137.6)
+			(xy 112 31.3) (xy 112.5 137.5)
 		)
 		(height 6.8)
@@
 		)
 		(gr_text "106.2"
-			(at 117.65 84.5 90)
+			(at 117.65 84.4 90)
 			(layer "Dwgs.User")
 			(effects

Commit message: Controlled Load Simulation
Other:
- board size 69.7 x 89.6 mm -> 67.6 x 103 mm
